File: t13-DFN10-prog-adapter.kicad_pcb (KiCad board)
At the start: 2 copper layers, 20.1 x 23.4 mm, 10 parts, among them P1 CONN_5, P2 CONN_5, P3 DFN10

Commit message: Tweaks.
Other:
- board text added: "ATtiny13 DFN10 programming adapter V0.10.b blog.spitzenpfeil.org 2014"
- board text removed: "ATtiny13 DFN10 programming adapter V0.10.a blog.spitzenpfeil.org 2014"

Commit message: Got the prototypes, adjusted internal cutouts.
Other:
- board text added: "ATtiny13 DFN10 programming adapter V0.10.c blog.spitzenpfeil.org 2014"
- board text removed: "ATtiny13 DFN10 programming adapter V0.10.b blog.spitzenpfeil.org 2014"
Changed lines of the file:
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@@
-(kicad_pcb (version 3) (host pcbnew "(2014-03-14 BZR 4750)-product")
+(kicad_pcb (version 3) (host pcbnew "(2014-04-04 BZR 4786)-product")
   (general
     (links 14)
@@
       (xy 0.82042 -0.95758) (xy 0.88392 -0.9398) (xy 0.889 -0.9398) (xy 0.9525 -0.93726)) (layer F.SilkS) (width 0.00254))
   )
-  (gr_text "ATtiny13 DFN10\nprogramming adapter\n\nV0.10.b\nblog.spitzenpfeil.org\n2014" (at 163.2712 101.5746 90) (layer B.SilkS)
+  (gr_text "ATtiny13 DFN10\nprogramming adapter\n\nV0.10.c\nblog.spitzenpfeil.org\n2014" (at 163.2712 101.5746 90) (layer B.SilkS)
     (effects (font (size 1 1) (thickness 0.25)) (justify mirror))
   )
@@
   (gr_line (start 155.956 89.916) (end 176.022 89.916) (angle 90) (layer Edge.Cuts) (width 0.1))
   (gr_line (start 155.956 113.284) (end 176.022 113.284) (angle 90) (layer Edge.Cuts) (width 0.1))
+  (segment (start 161.56 107.68) (end 157.48 111.76) (width 0.254) (layer F.Cu) (net 1))
+  (segment (start 161.56 103.1) (end 161.56 107.68) (width 0.254) (layer F.Cu) (net 1))
+  (segment (start 165.1 104.14) (end 157.48 111.76) (width 0.254) (layer B.Cu) (net 1))
   (segment (start 171.704 104.14) (end 165.1 104.14) (width 0.254) (layer B.Cu) (net 1))
-  (segment (start 165.1 104.14) (end 157.48 111.76) (width 0.254) (layer B.Cu) (net 1))
-  (segment (start 161.56 103.1) (end 161.56 107.68) (width 0.254) (layer F.Cu) (net 1))
-  (segment (start 161.56 107.68) (end 157.48 111.76) (width 0.254) (layer F.Cu) (net 1))
+  (segment (start 161.56 95.52) (end 157.48 91.44) (width 0.254) (layer F.Cu) (net 2))
+  (segment (start 161.56 100.1) (end 161.56 95.52) (width 0.254) (layer F.Cu) (net 2))
+  (segment (start 157.48 92.0496) (end 157.48 91.44) (width 0.254) (layer B.Cu) (net 2))
+  (segment (start 174.244 98.044) (end 173.3804 97.1804) (width 0.254) (layer F.Cu) (net 2))
+  (segment (start 173.3804 97.1804) (end 171.1452 97.1804) (width 0.254) (layer F.Cu) (net 2))
+  (segment (start 171.1452 97.1804) (end 166.878 101.4476) (width 0.254) (layer F.Cu) (net 2))
+  (via (at 166.878 101.4476) (size 0.889) (layers F.Cu B.Cu) (net 2))
+  (segment (start 166.878 101.4476) (end 157.48 92.0496) (width 0.254) (layer B.Cu) (net 2))
   (segment (start 174.244 99.06) (end 174.244 98.044) (width 0.254) (layer F.Cu) (net 2))
-  (segment (start 166.878 101.4476) (end 157.48 92.0496) (width 0.254) (layer B.Cu) (net 2))
-  (via (at 166.878 101.4476) (size 0.889) (layers F.Cu B.Cu) (net 2))
-  (segment (start 171.1452 97.1804) (end 166.878 101.4476) (width 0.254) (layer F.Cu) (net 2))
-  (segment (start 173.3804 97.1804) (end 171.1452 97.1804) (width 0.254) (layer F.Cu) (net 2))
-  (segment (start 174.244 98.044) (end 173.3804 97.1804) (width 0.254) (layer F.Cu) (net 2))
-  (segment (start 157.48 92.0496) (end 157.48 91.44) (width 0.254) (layer B.Cu) (net 2))
-  (segment (start 161.56 100.1) (end 161.56 95.52) (width 0.254) (layer F.Cu) (net 2))
-  (segment (start 161.56 95.52) (end 157.48 91.44) (width 0.254) (layer F.Cu) (net 2))
+  (segment (start 162.06 93.48) (end 160.02 91.44) (width 0.254) (layer F.Cu) (net 3))
+  (segment (start 162.06 100.1) (end 162.06 93.48) (width 0.254) (layer F.Cu) (net 3))
+  (segment (start 170.18 101.6) (end 160.02 91.44) (width 0.254) (layer B.Cu) (net 3))
   (segment (start 171.704 101.6) (end 170.18 101.6) (width 0.254) (layer B.Cu) (net 3))
-  (segment (start 170.18 101.6) (end 160.02 91.44) (width 0.254) (layer B.Cu) (net 3))
-  (segment (start 162.06 100.1) (end 162.06 93.48) (width 0.254) (layer F.Cu) (net 3))
-  (segment (start 162.06 93.48) (end 160.02 91.44) (width 0.254) (layer F.Cu) (net 3))
+  (segment (start 163.06 93.48) (end 165.1 91.44) (width 0.254) (layer F.Cu) (net 4))
+  (segment (start 163.06 100.1) (end 163.06 93.48) (width 0.254) (layer F.Cu) (net 4))
+  (segment (start 168.6306 99.06) (end 165.1 95.5294) (width 0.254) (layer B.Cu) (net 4))
+  (segment (start 165.1 95.5294) (end 165.1 91.44) (width 0.254) (layer B.Cu) (net 4))
   (segment (start 171.704 99.06) (end 168.6306 99.06) (width 0.254) (layer B.Cu) (net 4))
-  (segment (start 165.1 95.5294) (end 165.1 91.44) (width 0.254) (layer B.Cu) (net 4))
-  (segment (start 168.6306 99.06) (end 165.1 95.5294) (width 0.254) (layer B.Cu) (net 4))
-  (segment (start 163.06 100.1) (end 163.06 93.48) (width 0.254) (layer F.Cu) (net 4))
-  (segment (start 163.06 93.48) (end 165.1 91.44) (width 0.254) (layer F.Cu) (net 4))
+  (segment (start 163.56 107.68) (end 167.64 111.76) (width 0.254) (layer F.Cu) (net 5))
+  (segment (start 163.56 103.1) (end 163.56 107.68) (width 0.254) (layer F.Cu) (net 5))
+  (segment (start 174.244 105.156) (end 167.64 111.76) (width 0.254) (layer B.Cu) (net 5))
   (segment (start 174.244 104.14) (end 174.244 105.156) (width 0.254) (layer B.Cu) (net 5))
-  (segment (start 174.244 105.156) (end 167.64 111.76) (width 0.254) (layer B.Cu) (net 5))
-  (segment (start 163.56 103.1) (end 163.56 107.68) (width 0.254) (layer F.Cu) (net 5))
-  (segment (start 163.56 107.68) (end 167.64 111.76) (width 0.254) (layer F.Cu) (net 5))
+  (segment (start 163.56 95.52) (end 167.64 91.44) (width 0.254) (layer F.Cu) (net 6))
+  (segment (start 163.56 100.1) (end 163.56 95.52) (width 0.254) (layer F.Cu) (net 6))
+  (segment (start 174.244 101.6) (end 175.4632 100.3808) (width 0.254) (layer B.Cu) (net 6))
+  (segment (start 175.4632 100.3808) (end 175.4632 98.1842) (width 0.254) (layer B.Cu) (net 6))
+  (segment (start 175.4632 98.1842) (end 168.719 91.44) (width 0.254) (layer B.Cu) (net 6))
   (segment (start 168.719 91.44) (end 167.64 91.44) (width 0.254) (layer B.Cu) (net 6))
-  (segment (start 175.4632 98.1842) (end 168.719 91.44) (width 0.254) (layer B.Cu) (net 6))
-  (segment (start 175.4632 100.3808) (end 175.4632 98.1842) (width 0.254) (layer B.Cu) (net 6))
-  (segment (start 174.244 101.6) (end 175.4632 100.3808) (width 0.254) (layer B.Cu) (net 6))
-  (segment (start 163.56 100.1) (end 163.56 95.52) (width 0.254) (layer F.Cu) (net 6))
-  (segment (start 163.56 95.52) (end 167.64 91.44) (width 0.254) (layer F.Cu) (net 6))
+  (segment (start 162.06 109.72) (end 160.02 111.76) (width 0.254) (layer F.Cu) (net 7))
   (segment (start 162.06 103.1) (end 162.06 109.72) (width 0.254) (layer F.Cu) (net 7))
-  (segment (start 162.06 109.72) (end 160.02 111.76) (width 0.254) (layer F.Cu) (net 7))
+  (segment (start 163.06 109.72) (end 165.1 111.76) (width 0.254) (layer F.Cu) (net 9))
   (segment (start 163.06 103.1) (end 163.06 109.72) (width 0.254) (layer F.Cu) (net 9))
-  (segment (start 163.06 109.72) (end 165.1 111.76) (width 0.254) (layer F.Cu) (net 9))
   (zone (net 0) (net_name "") (layer F.Mask) (hatch full 0.508)
     (connect_pads (clearance 0.508))
